File: fZero.kicad_sch (KiCad schematic)
At the start: 53 parts, among them J1 Raspberry_Pi_2x20_SMD_Passthr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, J2 Conn_01x08_Pin, J3 USB_C_Receptacle_PowerOnly_6P, SW1 SW_Push_45deg, SW10 SW_Push_45deg, SW11 SW_Push_45deg, SW12 SW_Push_45deg, SW13 SW_Push_45deg, SW14 SW_Push_45deg, SW15 SW_Push_45deg, SW16 SW_Push_45deg, SW2 SW_Push_45deg, SW3 SW_Push_45deg, SW4 SW_Push_45deg, SW5 SW_Push_45deg, SW6 SW_Push_45deg, SW7 SW_Push_45deg, SW8 SW_Push_45deg, SW9 SW_Push_45deg, U1 ER_OLEDM0.91_1x-I2C, U2 BQ24074RGT

Commit message: nearly done! a bit more to go for the schematic
Parts:
- removed BT1: Battery_Cell, symbol Device:Battery_Cell
- added BT1: BH-18650-B1BA002, easyeda2kicad:BATTERY-SMD_18650-1S-L77.1-W20.7-1, symbol JLC_Parts:BH-18650-B1BA002
- added BZ1: Buzzer, symbol Device:Buzzer
- added C10, C8, C9: 22uF, symbol Device:C_Small
- added C6: 0.1uF, symbol Device:C_Small
- added C7: 10uF, symbol Device:C_Small
- added L1: 1uH, symbol Device:L
- added Q1: FS8205A_C908265, easyeda2kicad:SOT-23-6_L2.9-W1.6-P0.95-LS2.8-BR, symbol JLC_Parts:FS8205A_C908265
- added R10: 1.5K, symbol Device:R_Small
- added R11: 732K, symbol Device:R_Small
- added R12: 100K, symbol Device:R_Small
- added R3: 100, symbol Device:R_Small
- added SW17: Switch_Slide_RightAngle_CnK, PCM_fab:Switch_Slide_RightAngle_CnK_AYZ0102AGRLC_7.2x3mm, symbol PCM_fab:Switch_Slide_RightAngle_CnK
- added SW18: SW_Push, symbol Switch:SW_Push
- added TH1: Thermistor_NTC, symbol Device:Thermistor_NTC
- added U3: DW01A, Package_TO_SOT_SMD:SOT-23-6, symbol Battery_Management:DW01A
- added U4: TPS61022, Package_DFN_QFN:Texas_RWU0007A_VQFN-7_2x2mm_P0.5mm, symbol Converter_DCDC:TPS61022
- added U5: MAX17048, PCM_SparkFun-Semiconductor-Standard:DFN-8_2x2mm_P0.5mm_EP1.2x0.8mm, symbol PCM_SparkFun-IC-Power:MAX17048
- R1, R2: value R -> 5.1K
- R4, R5: value R_Small -> 1.5K
- R6, R7: value R_Small -> 1.2K
- R8: value R_Small -> 47K
- R9: value R_Small -> 4.3K
Connections:
- net +4V: now also C5.1, U2.2 (BAT), U2.3 (BAT), BT1.1, C7.2, L1.1, R3.1, SW17.2 (B), U4.7 (VIN), U5.2 (CELL), U5.3 (VDD)
- net DISPLAY_DC: no longer J1.22 (GPIO25)
- net GND: now also J1.14 (GND), J1.20 (GND), J1.25 (GND), J1.30 (GND), J1.34 (GND), J1.39 (GND), J1.6 (GND), J1.9 (GND), BT1.2, C10.1, C6.2, C7.1, Q1.1 (S1), Q1.3 (S2), R10.1, R12.2, SW18.2, TH1.2, U3.6 (GND), U4.1 (GND), U4.6 (MODE), U5.1 (CTG), U5.4 (GND), U5.6 (QSTRT), U5.9 (GND)
- net 5V: now reaches J1.2 (5V), J1.4 (5V)
- net 5V: now also C8.2, R11.1, U4.3 (VOUT)
- net SHUTTER_BTN: now reaches J1.7 (GCLK0/GPIO4)
- net SHUTTER_BTN: now also SW18.1
- net at U2.1 (TS): now also TH1.1
- net CHARGE_DISP_SCL renamed I2C0_SCL
- net I2C0_SCL: now also U5.7 (SCL)
- net CHARGE_DISP_SDA renamed I2C0_SDA
- net I2C0_SDA: now also U5.8 (SDA)
- new net: Q1.6 (G1), U3.1 (OD)
- new net: R10.2, U3.2 (CS)
- new net: Q1.4 (G2), U3.3 (OC)
- new net: C6.1, R3.2, U3.5 (VCC)
- new net: L1.2, U4.2 (SW)
- new net: R11.2, R12.1, U4.4 (FB)
- new net: SW17.1 (A), U4.5 (EN)
- new net: C10.2, C9.1
- new net: C8.1, C9.2
- new net: Q1.2 (D1/D2), Q1.5 (D1/D2)
- no-connect marks 0 -> 1
Other:
- note added: "Battery Protection"
- note added: "Boost Converter"
- note added: "Buzzer"
- note added: "Camera Shutter"
- note added: "Flash"
- note added: "Fuel Gauge"
- moved on the sheet: C3, C4, C5, D17, D18, R4, R5, R6, R7, R8, R9, U2

Commit message: finished PCB design, starting partialy sourcing parts
Parts:
- added C11: 47nF, Resistor_SMD:R_0201_0603Metric, symbol Device:C_Small
- added D19: LED, Connector_Wire:SolderWire-0.75sqmm_1x02_P4.8mm_D1.25mm_OD2.3mm, symbol Device:LED
- added D20: D, Diode_SMD:D_SOD-123, symbol Device:D
- added Q2: AO3400A, PCM_Package_TO_SOT_SMD_AKL:SOT-23, symbol PCM_Transistor_MOSFET_AKL:AO3400A
- added Q3: MMBT3904, PCM_Package_TO_SOT_SMD_AKL:SOT-23, symbol PCM_Transistor_BJT_AKL:MMBT3904
- added R13: 1.5K, symbol Device:R
- added R14: 100K, symbol Device:R
- added R15: 10K, symbol Device:R
- added R16: 0.82, symbol Device:R
- added R17: 100K, symbol Device:R_Small
- BT1: footprint easyeda2kicad:BATTERY-SMD_18650-1S-L77.1-W20.7-1 -> JLC_Parts:BATTERY-SMD_18650-1S-L77.1-W20.7-1
- BZ1: footprint (none) -> Buzzer_Beeper:Buzzer_12x9.5RM7.6
- C1, C4, C5: value C_Small -> 4.7uF; footprint (none) -> Resistor_SMD:R_0805_2012Metric; JLCPCB Part # (none) -> C1779
- C10, C8, C9: footprint (none) -> Resistor_SMD:R_1206_3216Metric; JLCPCB Part # (none) -> C5672
- C2: value C_Small -> 100nF; footprint (none) -> Resistor_SMD:R_0805_2012Metric; JLCPCB Part # (none) -> C1779
- C3: value C_Small -> 1uF; footprint (none) -> Resistor_SMD:R_0805_2012Metric; JLCPCB Part # (none) -> C1712
- C6: footprint (none) -> Resistor_SMD:R_0402_1005Metric; JLCPCB Part # (none) -> C1525
- C7: value 10uF -> 22uF; footprint (none) -> Resistor_SMD:R_1206_3216Metric; JLCPCB Part # (none) -> C5672
- D1, D10, D11, D12, D13, D14, D15, D16, D2, D3, D4, D5, D6, D7, D8, D9: footprint (none) -> Diode_SMD:D_SOD-123; JLCPCB Part # (none) -> C81598
- J3: footprint (none) -> Connector_USB:USB_C_Receptacle_GCT_USB4125-xx-x-0190_6P_TopMnt_Horizontal
Connections:
- net DISPLAY_RST is gone; now on net DISPLAY_RESET: J1.28 (ID_SC/GPIO1)
- net +4V: no longer BT1.1, C4.1, C5.1, C7.2, L1.1, R3.1, R4.2, R5.2, SW17.2 (B), U2.10 (OUT), U2.11 (OUT), U2.2 (BAT), U2.3 (BAT), U2.5 (EN2), U4.7 (VIN), U5.3 (VDD)
- net 5V: now also C11.2, D19.2 (A)
- net COLUMN2: now also D10.1 (K), D12.1 (K); no longer D13.1 (K), D15.1 (K)
- net COLUMN3: now also D13.1 (K), D15.1 (K); no longer D10.1 (K), D12.1 (K)
- net GND: now also BZ1.2 (-), C11.1, D20.2 (A), Q3.2 (E), R14.2, R16.2; no longer BT1.2, C6.2, Q1.1 (S1), U3.6 (GND)
- net PWR_3V3: now also J1.1 (3V3), J1.17 (3V3)
- net at D13.2 (A): now also SW10.2; no longer SW13.2
- net at U4.5 (EN): now also R17.1; no longer SW17.1 (A)
- net at SW11.2: now also D10.2 (A); no longer D11.2 (A)
- net BUZZER: now reaches BZ1.1 (+)
- net at SW12.2: now also D14.2 (A); no longer D12.2 (A)
- net CAMERA_FLASH: now reaches J1.11 (GPIO17)
- net CAMERA_FLASH: now also D20.1 (K), R14.1, R15.1
- net at D15.2 (A): now also SW14.2; no longer SW15.2
- new net: Q2.1 (G), Q3.3 (C), R15.2
- new net: BT1.2, C6.2, Q1.1 (S1), U3.6 (GND)
- new net: D19.1 (K), R13.1
- new net: Q2.3 (D), R13.2
- new net: Q2.2 (S), Q3.1 (B), R16.1
- new net: R17.2, SW17.1 (A)
- new net: D12.2 (A), SW15.2
- new net: D11.2 (A), SW13.2
- new net +BATT: BT1.1, C5.1, R3.1, U2.2 (BAT), U2.3 (BAT), U5.3 (VDD)
- new net VCC: C4.1, C7.2, L1.1, R4.2, R5.2, SW17.2 (B), U2.10 (OUT), U2.11 (OUT), U2.5 (EN2), U4.7 (VIN)
- no-connect marks 1 -> 8
Other:
- note added: "Active Buzzer"
- note added: "Battery & Protection"
- note added: "Flash (LH31D)"
- note removed: "Battery Protection"
- note removed: "Buzzer"
- note removed: "Flash"
- moved on the sheet: C1, C10, C2, C7, C8, C9, J3, L1, R1, R11, R12, R2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
